Commit message: small adjustments to urdf

File: urdf/ur5e_description/ur5e.urdf.xacro (robot description, xacro)
@@ -330,7 +330,7 @@
       <!-- added box for collision detection for qbhand + box-->
       <visual>
-        <origin xyz="0 0 0.12" rpy="0 0 0"/>
-        <geometry>
-          <box size="0.056  0.17 0.24"/>
+        <origin xyz="-0.02 0 0.10" rpy="0 0 ${-pi/2.0}"/>
+        <geometry>
+          <box size="0.056  0.191 0.24"/>
         </geometry>
         <material name="blue">
@@ -339,6 +339,7 @@
       </visual>
       <collision>
-        <geometry>
-          <box size="0.056  0.17 0.24"/>
+        <origin xyz="-0.02 0 0.10" rpy="0 0 ${-pi/2.0}"/>
+        <geometry>
+          <box size="0.056  0.191 0.24"/>
         </geometry>
       </collision>

Commit message: rough adjustments to urdf

File: urdf/ur5e_description/ur5e.urdf.xacro (robot description, xacro)
@@ -330,21 +330,21 @@
       <!-- added box for collision detection for qbhand + box-->
       <visual>
-        <origin xyz="-0.02 0 0.10" rpy="0 0 ${-pi/2.0}"/>
-        <geometry>
-          <box size="0.056  0.191 0.24"/>
-        </geometry>
-        <material name="blue">
-          <color rgba="1 0 .8 1" />
-        </material>
-      </visual>
-      <collision>
-        <origin xyz="-0.02 0 0.10" rpy="0 0 ${-pi/2.0}"/>
-        <geometry>
-          <box size="0.056  0.191 0.24"/>
+        <origin xyz="0.0 0.0225 0.0" rpy="0 0 ${-pi/2.0}"/>
+        <geometry>
+          <box size="0.135  0.18 0.17"/>
+        </geometry>
+        <material name="pink">
+          <color rgba="1 0 .8 0.5" />
+        </material>
+      </visual>
+      <collision>
+        <origin xyz="0.0 0.0375 0.08" rpy="0 0 ${-pi/2.0}"/>
+        <geometry>
+          <box size="0.135  0.18 0.17"/>
         </geometry>
       </collision>
     </link>
     <joint name="${prefix}wrist_3_link-tool0_fixed_joint" type="fixed">
-      <origin xyz="0 0 0.06" rpy="0 0 0" />
+      <origin xyz="0 0.0225 0.145" rpy="0 0 0" />
       <parent link="${prefix}wrist_3_link" />
       <child link="${prefix}tool0" />

Commit message: new values for tool0 position in urdf

File: urdf/ur5e_description/ur5e.urdf.xacro (robot description, xacro)
@@ -346,5 +346,5 @@
     </link>
     <joint name="${prefix}wrist_3_link-tool0_fixed_joint" type="fixed">
-      <origin xyz="0 0.0225 0.145" rpy="0 0 0" />
+      <origin xyz="0.00973 0.03636 0.12945" rpy="0 0 0" />
       <parent link="${prefix}wrist_3_link" />
       <child link="${prefix}tool0" />

Commit message: new factors for newjointspeed and tests

File: urdf/ur5e_description/ur5e.urdf.xacro (robot description, xacro)
@@ -346,5 +346,5 @@
     </link>
     <joint name="${prefix}wrist_3_link-tool0_fixed_joint" type="fixed">
-      <origin xyz="0.00973 0.03636 0.12945" rpy="0 0 0" />
+      <origin xyz="0.01138 0.1141 0.14719" rpy="0 0 0" />
       <parent link="${prefix}wrist_3_link" />
       <child link="${prefix}tool0" />
